Commit message: Update omxa.xacro

File: 로봇팔/omxa_description/urdf/omxa.xacro (robot description, xacro)
@@ -469,5 +469,5 @@
   <parent link="brk8_1"/>
   <child link="camera_link"/>
-  <origin xyz="0.0115 0.03045 0.0458" rpy="0 0 0"/>
+  <origin xyz="-0.03266 0.02736 0.0458" rpy="0 0 0"/>
 </joint>
 <link name="camera_color_optical_frame"/>
